File: Hardware/DesignFiles/KiCAD/Masjid2.kicad_pcb (KiCad board)
At the start: 2 copper layers, 76 x 56.5 mm, 65 parts, among them J1 12V_CONNx2, J2 LIGHT_SWITCH_CONNx2, J3 ISP_CONNx6, J4 LED_STRIP_12V_CONNx2, J5 FTDI_CONNx6, J6 SPEAKER_CONNx2, J7 DS3231_CONNx4, Q1 IRLZ44N, SW1 RST_BTN, U1 AMS1117-3.3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

Commit message: ready for stasis build review
Parts:
- removed R1: 1R, Resistor_SMD:R_0805_2012Metric
- removed REF** (x4): MountingHole_1.5mm_No_Courtyard, MountingHole:MountingHole_2.1mm
- removed TP1: PWM_TP, TestPoint:TestPoint_Pad_2.0x2.0mm
- removed TP2: SPEAKER_TP, TestPoint:TestPoint_Pad_2.0x2.0mm
- removed TP4: PD7_TP, TestPoint:TestPoint_Pad_2.0x2.0mm
- removed U5: ATmega328P-A, Package_QFP:TQFP-32_7x7mm_P0.8mm
- added PD7: PD7_TP, TestPoint:TestPoint_Pad_2.0x2.0mm, F.Cu at (150.2, 109.8)
- added PWM: PWM_TP, TestPoint:TestPoint_Pad_2.0x2.0mm, F.Cu at (156.0, 96.0)
- added SPKR: SPEAKER_TP, TestPoint:TestPoint_Pad_2.0x2.0mm, F.Cu at (171.9, 117.3)
- added U6: ATmega328P-P, Package_DIP:DIP-28_W7.62mm, F.Cu at (119.5, 106.6)
- moved R6 264.8 mm to (164.7, 109.5), turned to 180 degrees
- moved C14 264.3 mm to (168.6, 108.3), turned to -90 degrees
- moved C9 262.7 mm to (170.2, 104.0), turned to 55 degrees
- moved Y1 261.9 mm to (144.7, 110.8), turned to 180 degrees
- moved C17 261.9 mm to (145.7, 115.0), turned to 180 degrees
- moved J3 258.2 mm to (164.1, 77.3), turned to -90 degrees
- moved C15 257.9 mm to (138.7, 115.0), turned to 180 degrees
- moved C18 254.8 mm to (162.3, 114.5), turned to 180 degrees
- moved C10 253.6 mm to (134.3, 109.2), turned to 175 degrees
- moved C12 248.4 mm to (170.2, 111.8)
- moved C8 247.1 mm to (155.8, 87.0), turned to -90 degrees
- moved R10 246.4 mm to (135.0, 75.8), turned to 0 degrees
- moved R12 246.3 mm to (115.6, 106.5), turned to 180 degrees
- moved J7 246.2 mm to (135.9, 78.3)
- moved U4 246.0 mm to (161.3, 101.3), turned to 0 degrees
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Connections:
- C4 pad 2: Net-(C4-Pad2) -> GND
- R14 pad 2: /PD5 -> /PC3
Routing:
- net +3.3V: track 228.0 -> 163.9 mm, vias 7 -> 9
- net +12V: track 81.1 -> 140.5 mm, vias 1 -> 5
- net /FTDI_DTR: track 51.8 -> 8.66 mm
- net /PD1_TXD: track 48.9 -> 11.5 mm, vias 1 -> 0
- net Net-(U4--): track 47.7 -> 13.1 mm, vias 0 -> 1
- net /PD0_RXD: track 40.0 -> 11.2 mm, vias 1 -> 2
- net /PC6_RST: track 63.0 -> 85.1 mm, vias 0 -> 3
- net Net-(U4-+): track 27.8 -> 6.78 mm, vias 0 -> 1
- net /PB2_CS: track 27.6 -> 8.68 mm, vias 3 -> 1
- net Net-(C12-Pad1): track 33.0 -> 16.8 mm, vias 0 -> 3
- net /PD5: track 15.6 -> 0.00 mm
- net /PC5_SCL: track 26.8 -> 41.5 mm
- net GND: track 15.8 -> 2.34 mm, vias 11 -> 14
- net +5V: track 44.6 -> 31.7 mm, vias 0 -> 4
- net /PB3_MOSI: track 46.1 -> 34.3 mm
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Other:
- board size 76 x 56.5 mm -> 76 x 45.2 mm
- board text added: "26/06/03"
- board text added: "3V3"
- board text added: "DTR"
- board text added: "GND"
- board text added: "MISO"
- board text added: "MOSI"
- board text added: "RST"
- board text added: "RXD"
- board text added: "SCK"
- board text added: "TXD"
