File: Hardware/DesignFiles/KiCAD/Masjid2.kicad_sch (KiCad schematic)
At the start: 61 parts, among them J1 12V_CONNx2, J2 LIGHT_SWITCH_CONNx2, J3 ISP_CONNx6, J4 LED_STRIP_12V_CONNx2, J5 FTDI_CONNx6, J6 SPEAKER_CONNx2, J7 DS3231_CONNx4, Q1 IRLZ44N, SW1 RST_BTN, U1 AMS1117-3.3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

Commit message: ready for stasis build review
Parts:
- removed R1: 1R, Resistor_SMD:R_0805_2012Metric, symbol Device:R_Small
- removed U5: ATmega328P-A, Package_QFP:TQFP-32_7x7mm_P0.8mm, symbol MCU_Microchip_ATmega:ATmega328P-A
- added U6: ATmega328P-P, Package_DIP:DIP-28_W7.62mm, symbol MCU_Microchip_ATmega:ATmega328P-P
Connections:
- net +3.3V: now also U6.20 (AVCC), U6.7 (VCC)
- net GND: now also C4.2, U6.22 (GND), U6.8 (GND)
- net PB0: now also U6.14 (PB0)
- net PB1_PWM: now also U6.15 (PB1)
- net PB2_CS: now also U6.16 (PB2)
- net PB3_MOSI: now also U6.17 (PB3)
- net PB4_MISO: now also U6.18 (PB4)
- net PB5_SCK: now also U6.19 (PB5)
- net PC0: now also U6.23 (PC0)
- net PC1: now also U6.24 (PC1)
- net PC2: now also U6.25 (PC2)
- net PC3: now also R14.2, U6.26 (PC3)
- net PC4_SDA: now also U6.27 (PC4)
- net PC5_SCL: now also U6.28 (PC5)
- net PC6_RST: now also U6.1 (~{RESET}/PC6)
- net PD0_RXD: now also U6.2 (PD0)
- net PD1_TXD: now also U6.3 (PD1)
- net PD2: now also U6.4 (PD2)
- net PD3: now also U6.5 (PD3)
- net PD4: now also U6.6 (PD4)
- net PD5: now also U6.11 (PD5); no longer R14.2
- net PD6: now also U6.12 (PD6)
- net PD7: now also U6.13 (PD7)
- net at C15.1, Y1.2: now also U6.9 (XTAL1/PB6)
- net at C17.2, Y1.1: now also U6.10 (XTAL2/PB7)
- no-connect marks 10 -> 8
Other:
- note added: "X"
- moved on the sheet: C7, R12, U3
